File: nrf-rust-feather.kicad_pcb (KiCad board)
At the start: 4 copper layers, 51 parts, among them J101 Conn_01x12, J102 Conn_01x16, J103 USB_C_Receptacle_USB2.0, U101 nRF52840, U102 LSM6DSM, U103 USB2422, U104 STM32F042K6Tx, U105 MIC5259, Y101 32 MHz, Y102 24 MHz

Commit message: Some layout, more parts
Parts:
- added C130: 18p, passive:C_0402, F.Cu at (163.4, 84.6)
- added C131: 18p, passive:C_0402, F.Cu at (163.4, 86.6)
- added D101: LED_Small, LED_SMD:LED_0402_1005Metric, F.Cu at (108.0, 78.5)
- added D102: LED_Small, LED_SMD:LED_0402_1005Metric, F.Cu at (108.0, 80.5)
- added D103: LED_Small, LED_SMD:LED_0402_1005Metric, F.Cu at (108.0, 82.5)
- added H101: MountingHole_Pad, MountingHole:MountingHole_2.5mm_Pad, F.Cu at (129.5, 78.7)
- added H102: MountingHole_Pad, MountingHole:MountingHole_2.5mm_Pad, F.Cu at (129.5, 96.5)
- added J104: QWIIC, connectors:SM04B-SRSS-TB, F.Cu at (178.0, 95.6)
- added R110: 47k, passive:R_0402, F.Cu at (110.8, 78.4)
- added R111: 47k, passive:R_0402, F.Cu at (110.8, 80.3)
- added R112: 1k, passive:R_0402, F.Cu at (107.6, 84.4)
- added R113: 1k, passive:R_0402, F.Cu at (113.4, 78.4)
- added R114: 1k, passive:R_0402, F.Cu at (110.8, 82.1)
- added SW101: SW_SPST, pushbuttons:SW_SPST_KMR2, F.Cu at (103.0, 79.8)
- added SW102: SW_SPST, pushbuttons:SW_SPST_KMR2, F.Cu at (103.0, 84.5)
- added Y103: 32kHz, Crystal:Crystal_SMD_3215-2Pin_3.2x1.5mm, F.Cu at (165.0, 85.6)
- moved J102 79.5 mm to (172.7, 97.8), turned to 90 degrees
- moved C102 78.4 mm to (176.9, 86.4), turned to 270 degrees
- moved J101 75.8 mm to (172.7, 77.5), turned to 90 degrees
- moved C107 75.5 mm to (174.3, 86.4), turned to 270 degrees
- moved L101 70.7 mm to (175.6, 86.8), turned to 180 degrees
- moved AE101 68.9 mm to (186.0, 85.4), turned to 90 degrees
- moved Y101 67.5 mm to (173.0, 82.6), turned to 180 degrees
- moved U101 58.2 mm to (170.0, 87.6)
- moved U105 49.0 mm to (139.5, 92.5)
- moved U104 47.9 mm to (150.5, 84.1), turned to 180 degrees
- moved C129 45.4 mm to (142.0, 92.5), turned to 270 degrees
- moved J103 44.3 mm to (129.5, 87.6), turned to 270 degrees
- moved C125 38.7 mm to (137.0, 92.5), turned to 90 degrees
- moved U103 37.2 mm to (140.0, 85.6), turned to 180 degrees
Connections:
- U101 pad A12: Net-(U101-PadA12) -> BTN1
- U101 pad AD22: Net-(U101-PadAD22) -> SWO
- U101 pad B13: Net-(U101-PadB13) -> BTN2
- U101 pad J1: Net-(U101-PadJ1) -> LED1
- U101 pad K2: Net-(U101-PadK2) -> LED2
- U101 pad L1: Net-(U101-PadL1) -> LED3
- U101 pad W24: Net-(U101-PadW24) -> QWIIC_SDA
- U101 pad Y23: Net-(U101-PadY23) -> QWIIC_SCL
- U104 pad 9: Net-(U104-Pad9) -> SWO
Routing:
- net Net-(AE101-Pad1): track 0.00 -> 10.0 mm
- net GND: track 0.00 -> 8.46 mm, vias 9 -> 0
- net Net-(C107-Pad2): track 0.00 -> 2.62 mm
- net RESET: track 0.00 -> 1.79 mm, vias 0 -> 1
Other:
- board outline added: 60.5 x 22.9 mm

Commit message: Basic layout
Parts:
- removed C106: DNP, passive:C_0402
- removed C130, C131: 18p, passive:C_0402
- removed Y103: 32kHz, Crystal:Crystal_SMD_3215-2Pin_3.2x1.5mm
- moved C108 81.6 mm to (178.7, 84.2)
- moved C117 76.5 mm to (174.0, 92.3), turned to 90 degrees
- moved C101 75.7 mm to (181.8, 86.4), turned to 270 degrees
- moved U102 75.1 mm to (172.5, 81.1), turned to 180 degrees
- moved C104 75.0 mm to (179.4, 82.6), turned to 270 degrees
- moved C113 74.7 mm to (176.7, 91.9)
- moved C110 70.4 mm to (178.7, 85.1)
- moved C116 70.1 mm to (175.1, 82.6), turned to 270 degrees
- moved C109 69.2 mm to (178.7, 88.6)
- moved C105 69.0 mm to (176.0, 82.3), turned to 90 degrees
- moved C103 68.4 mm to (169.7, 85.0), turned to 90 degrees
- moved C118 68.0 mm to (171.6, 79.1), turned to 180 degrees
- moved C114 65.9 mm to (170.1, 92.1)
- moved SW102 62.8 mm to (165.5, 90.1)
- moved SW101 62.7 mm to (165.5, 85.1)
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Connections:
- U101 pad A10: Net-(U101-PadA10) -> IMU_CS
- U101 pad A12: BTN1 -> IMU_CLK
- U101 pad A14: IMU_INT2 -> IMU_SDI
- U101 pad A16: IMU_CS -> IMU_SDO
- U101 pad A20: IMU_SDO -> IMU_INT1
- U101 pad A8: Net-(U101-PadA8) -> IMU_INT2
- U101 pad B13: BTN2 -> Net-(U101-PadB13)
- U101 pad B15: IMU_INT1 -> Net-(U101-PadB15)
- U101 pad B17: IMU_CLK -> Net-(U101-PadB17)
- U101 pad B19: IMU_SDI -> Net-(U101-PadB19)
- U101 pad F2: Net-(C131-Pad1) -> BTN1
- U101 pad G1: Net-(U101-PadG1) -> BTN2
- U101 pad K2: LED2 -> Net-(U101-PadK2)
- U101 pad L1: LED3 -> LED2
- U101 pad N1: Net-(U101-PadN1) -> LED3
- U101 pad W24: QWIIC_SDA -> QWIIC_SCL
- U101 pad Y23: QWIIC_SCL -> QWIIC_SDA
Routing:
- net VUSB: track 0.00 -> 46.2 mm
- net SWDIO: track 0.00 -> 44.5 mm, vias 0 -> 2
- net RESET: track 1.79 -> 38.9 mm, vias 1 -> 2
- net +3V3: track 0.00 -> 36.3 mm, vias 0 -> 20
- net SWCLK: track 0.00 -> 36.0 mm, vias 0 -> 2
- net D1+: track 0.00 -> 34.0 mm, vias 0 -> 2
- net D1-: track 0.00 -> 33.1 mm, vias 0 -> 2
- net SWO: track 0.00 -> 33.1 mm, vias 0 -> 2
- net LED3: track 0.00 -> 15.2 mm, vias 0 -> 2
- net LED1: track 0.00 -> 13.3 mm, vias 0 -> 2
- net LED2: track 0.00 -> 13.1 mm, vias 0 -> 2
- net BTN1: track 0.00 -> 12.5 mm
- net /CC1: track 0.00 -> 11.4 mm
- net BTN2: track 0.00 -> 10.8 mm
- net Net-(FB101-Pad1): track 0.00 -> 10.6 mm, vias 0 -> 2
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- added copper zone on In2.Cu, net +3V3
- added copper zone on B.Cu, net GND
- added copper zone on F.Cu, net GND
- added copper zone on In1.Cu, net GND
