File: nrf-rust-feather.sch (KiCad schematic (older format))
At the start: 51 parts, among them J101 Conn_01x12, J102 Conn_01x16, J103 USB_C_Receptacle_USB2.0, U101 nRF52840, U102 LSM6DSM, U103 USB2422, U104 STM32F042K6Tx, U105 MIC5259, Y101 32 MHz, Y102 24 MHz

Commit message: Some layout, more parts
Parts:
- added C130, C131: 18p, passive:C_0402, symbol Device:C_Small
- added D101, D102, D103: LED_Small, LED_SMD:LED_0402_1005Metric, symbol Device:LED_Small
- added H101, H102: MountingHole_Pad, MountingHole:MountingHole_2.5mm_Pad, symbol Mechanical:MountingHole_Pad
- added J104: QWIIC, connectors:SM04B-SRSS-TB, symbol connectors:Conn_01x04
- added R110, R111: 47k, passive:R_0402, symbol Device:R_Small
- added R112, R113, R114: 1k, passive:R_0402, symbol Device:R_Small
- added SW101, SW102: SW_SPST, pushbuttons:SW_SPST_KMR2, symbol switches:SW_SPST
- added Y103: 32kHz, Crystal:Crystal_SMD_3215-2Pin_3.2x1.5mm, symbol Device:Crystal_Small
Connections:
- net +3V3: now also J104.2 (Pin_2), R110.2, R111.2
- net GND: now also C130.2, C131.2, D101.1 (K), D102.1 (K), D103.1 (K), H101.1, H102.1, J104.0 (Mechanical), J104.1 (Pin_1), SW101.2 (B), SW102.2 (B)
- net BTN1: now reaches U101.A12 (AIN0/P0.02)
- net BTN1: now also R110.1, SW101.1 (A)
- net SWO: now reaches U101.AD22 (TRACEDATA0/P1.00)
- net SWO: now also U104.9 (PA3)
- net BTN2: now reaches U101.B13 (AIN1/P0.03)
- net BTN2: now also R111.1, SW102.1 (A)
- net at U101.D2 (XL1/P0.00): now also C130.1, Y103.1
- net at U101.F2 (XL2/P0.01): now also C131.1, Y103.2
- net LED1: now reaches U101.J1 (AIN2/P0.04)
- net LED1: now also R112.1
- net LED2: now reaches U101.K2 (AIN3/P0.05)
- net LED2: now also R113.1
- net LED3: now reaches U101.L1 (P0.06)
- net LED3: now also R114.1
- net QWIIC_SDA: now reaches U101.W24 (P1.02)
- net QWIIC_SDA: now also J104.3 (Pin_3)
- net QWIIC_SCL: now reaches U101.Y23 (P1.01)
- net QWIIC_SCL: now also J104.4 (Pin_4)
- new net: D101.2 (A), R112.2
- new net: D102.2 (A), R113.2
- new net: D103.2 (A), R114.2
- no-connect marks 29 -> 28

Commit message: Basic layout
Parts:
- removed C106: DNP, passive:C_0402, symbol Device:C_Small
- removed C130, C131: 18p, passive:C_0402, symbol Device:C_Small
- removed Y103: 32kHz, Crystal:Crystal_SMD_3215-2Pin_3.2x1.5mm, symbol Device:Crystal_Small
Connections:
- net BTN1: now also U101.F2 (XL2/P0.01); no longer U101.A12 (AIN0/P0.02)
- net BTN2: now also U101.G1 (P0.26); no longer U101.B13 (AIN1/P0.03)
- net IMU_CLK: now also U101.A12 (AIN0/P0.02); no longer U101.B17 (P1.12)
- net IMU_CS: now also U101.A10 (AIN5/P0.29); no longer U101.A16 (P1.13)
- net IMU_INT1: now also U101.A20 (P1.10); no longer U101.B15 (P1.14)
- net IMU_INT2: now also U101.A8 (AIN7/P0.31); no longer U101.A14 (P1.15)
- net IMU_SDI: now also U101.A14 (P1.15); no longer U101.B19 (P1.11)
- net IMU_SDO: now also U101.A16 (P1.13); no longer U101.A20 (P1.10)
- net LED2: now also U101.L1 (P0.06); no longer U101.K2 (AIN3/P0.05)
- net LED3: now also U101.N1 (P0.08); no longer U101.L1 (P0.06)
- net QWIIC_SCL: now also U101.W24 (P1.02); no longer U101.Y23 (P1.01)
- net QWIIC_SDA: now also U101.Y23 (P1.01); no longer U101.W24 (P1.02)
- no-connect marks 28 -> 29
Changed lines of the file:
@@
-$EndComp
-$Comp
-L Device:C_Small C106
-U 1 1 5F058379
-P 2100 1400
-F 0 "C106" H 2008 1354 50  0000 R CNN
-F 1 "DNP" H 2008 1445 50  0000 R CNN
-F 2 "passive:C_0402" H 2100 1400 50  0001 C CNN
-F 3 "~" H 2100 1400 50  0001 C CNN
-	1    2100 1400
-	-1   0    0    1
 $EndComp
 $Comp
@@
 $EndComp
 $Comp
-L power:GND #PWR0107
-U 1 1 5F06114B
-P 2100 1300
-F 0 "#PWR0107" H 2100 1050 50  0001 C CNN
-F 1 "GND" V 2105 1172 50  0001 R CNN
-F 2 "" H 2100 1300 50  0001 C CNN
-F 3 "" H 2100 1300 50  0001 C CNN
-	1    2100 1300
-	-1   0    0    1
-$EndComp
-$Comp
 L power:GND #PWR0110
 U 1 1 5F061466
@@
 Wire Wire Line
 	3100 1800 3100 2350
-Wire Wire Line
-	3000 1900 2100 1900
-Wire Wire Line
-	2100 1900 2100 1500
-Wire Wire Line
-	3000 1900 3000 2350
 Wire Wire Line
 	2900 2000 1750 2000
@@
 Wire Wire Line
 	3150 9100 2950 9100
+Text GLabel 5150 7150 2    50   Input ~ 0
+IMU_SDO
 Text GLabel 5150 6850 2    50   Input ~ 0
-IMU_SDO
-Text GLabel 5150 7250 2    50   Input ~ 0
 IMU_INT1
-Text GLabel 5150 7150 2    50   Input ~ 0
+Text GLabel 5150 5450 2    50   Input ~ 0
 IMU_CS
-Text GLabel 5150 7050 2    50   Input ~ 0
+Text GLabel 5150 2850 2    50   Input ~ 0
 IMU_CLK
-Text GLabel 5150 6950 2    50   Input ~ 0
+Text GLabel 5150 7350 2    50   Input ~ 0
 IMU_SDI
-Text GLabel 5150 7350 2    50   Input ~ 0
+Text GLabel 5150 5650 2    50   Input ~ 0
 IMU_INT2
 Wire Wire Line
 	5000 6850 5150 6850
 Wire Wire Line
-	5000 6950 5150 6950
-Wire Wire Line
-	5000 7050 5150 7050
-Wire Wire Line
 	5000 7150 5150 7150
-Wire Wire Line
-	5000 7250 5150 7250
 Wire Wire Line
 	5000 7350 5150 7350
@@
 	1    0    0    -1
 $EndComp
+Text GLabel 5150 5950 2    50   Input ~ 0
+QWIIC_SDA
 Text GLabel 5150 6050 2    50   Input ~ 0
-QWIIC_SDA
-Text GLabel 5150 5950 2    50   Input ~ 0
 QWIIC_SCL
 Wire Wire Line
@@
 Text GLabel 8050 7300 0    50   Input ~ 0
 LED3
-Text GLabel 5150 2850 2    50   Input ~ 0
+Text GLabel 5150 5150 2    50   Input ~ 0
+BTN2
+Text GLabel 5150 2750 2    50   Input ~ 0
 BTN1
-Text GLabel 5150 2950 2    50   Input ~ 0
-BTN2
 Text GLabel 5150 3050 2    50   Input ~ 0
 LED1
-Text GLabel 5150 3150 2    50   Input ~ 0
+Text GLabel 5150 3250 2    50   Input ~ 0
 LED2
-Text GLabel 5150 3250 2    50   Input ~ 0
+Text GLabel 5150 3450 2    50   Input ~ 0
 LED3
 Wire Wire Line
 	5000 2850 5150 2850
 Wire Wire Line
-	5000 2950 5150 2950
-Wire Wire Line
 	5000 3050 5150 3050
 Wire Wire Line
-	5000 3150 5150 3150
+	5000 3450 5150 3450
 Wire Wire Line
 	5000 3250 5150 3250
-$Comp
-L Device:Crystal_Small Y103
-U 1 1 5F673104
-P 5250 2400
-F 0 "Y103" V 5204 2488 50  0000 L CNN
-F 1 "32kHz" V 5295 2488 50  0000 L CNN
-F 2 "Crystal:Crystal_SMD_3215-2Pin_3.2x1.5mm" H 5250 2400 50  0001 C CNN
-F 3 "~" H 5250 2400 50  0001 C CNN
-F 4 "FC-135 32.7680KA-AC0" H 5250 2400 50  0001 C CNN "MPN"
-	1    5250 2400
-	0    1    1    0
-$EndComp
-$Comp
-L Device:C_Small C130
-U 1 1 5F678F43
-P 5700 2200
-F 0 "C130" V 5471 2200 50  0000 C CNN
-F 1 "18p" V 5562 2200 50  0000 C CNN
-F 2 "passive:C_0402" H 5700 2200 50  0001 C CNN
-F 3 "~" H 5700 2200 50  0001 C CNN
-	1    5700 2200
-	0    -1   -1   0
-$EndComp
-$Comp
-L Device:C_Small C131
-U 1 1 5F678F49
-P 5700 2600
-F 0 "C131" V 5471 2600 50  0000 C CNN
-F 1 "18p" V 5562 2600 50  0000 C CNN
-F 2 "passive:C_0402" H 5700 2600 50  0001 C CNN
-F 3 "~" H 5700 2600 50  0001 C CNN
-	1    5700 2600
-	0    -1   -1   0
-$EndComp
-$Comp
-L power:GND #PWR0172
-U 1 1 5F678F4F
-P 5800 2600
-F 0 "#PWR0172" H 5800 2350 50  0001 C CNN
-F 1 "GND" V 5805 2472 50  0001 R CNN
-F 2 "" H 5800 2600 50  0001 C CNN
-F 3 "" H 5800 2600 50  0001 C CNN
-	1    5800 2600
-	0    -1   -1   0
-$EndComp
-$Comp
-L power:GND #PWR0173
-U 1 1 5F678F55
-P 5800 2200
-F 0 "#PWR0173" H 5800 1950 50  0001 C CNN
-F 1 "GND" V 5805 2072 50  0001 R CNN
-F 2 "" H 5800 2200 50  0001 C CNN
-F 3 "" H 5800 2200 50  0001 C CNN
-	1    5800 2200
-	0    -1   -1   0
-$EndComp
-Wire Wire Line
-	5600 2200 5250 2200
-Wire Wire Line
-	5250 2200 5250 2300
-Wire Wire Line
-	5600 2600 5250 2600
-Wire Wire Line
-	5250 2600 5250 2500
-Wire Wire Line
-	5250 2600 5250 2750
-Wire Wire Line
-	5250 2750 5000 2750
-Connection ~ 5250 2600
-Wire Wire Line
-	5250 2200 5100 2200
-Wire Wire Line
-	5100 2200 5100 2650
-Wire Wire Line
-	5100 2650 5000 2650
-Connection ~ 5250 2200
+Wire Wire Line
+	3000 2300 3000 2350
+NoConn ~ 3000 2350
+Wire Wire Line
+	5150 5650 5000 5650
+Wire Wire Line
+	5000 5450 5150 5450
+Wire Wire Line
+	5150 5150 5000 5150
+Wire Wire Line
+	5000 2750 5150 2750
 $EndSCHEMATC
